Commit message: start of ur5e on slede

File: robo_inspecto_launch/urdf/frame.urdf.xacro (robot description, xacro)
@@ -1,35 +1,24 @@
 <?xml version="1.0"?>
 <robot xmlns:xacro="http://www.ros.org/wiki/xacro" name="frame">
-<xacro:include filename="macro.urdf.xacro" />
-<link name="frame_link">
     <xacro:property name="frame_length" value="1" />
     <xacro:property name="frame_width" value="0.3" />
-    <xacro:property name="frame_height" value="0.12" />
-    <visual>
-        <origin rpy="0 0 ${pi/2}"/>
-        <geometry>
-            <mesh filename="package://robo_inspecto_launch/meshes/frame.stl"/>
-        </geometry>
-    </visual>
-    <collision>
-        <geometry>
-            <box size="${frame_length} ${frame_width} ${frame_height}" />
-        </geometry>
-    </collision>
-</link>
-<!-- link frame to base -->
-<link name="base_link">
-</link>
-<joint name="base_to_frame" type="fixed">
-    <parent link="base_link" />
-    <child link="frame_link" />
-    <origin xyz="0 0 0" />
-</joint>
-<xacro:include filename="slede.urdf.xacro" />
-<!-- connect slede to frame -->
-<joint name="frame_to_slede" type="fixed">
-    <parent link="frame_link" />
-    <child link="base_plate_link" />
-    <origin xyz="0 0 0.12" />
-</joint>
+    <xacro:property name="frame_height" value="0.1125" />
+    <material name="light_grey">
+        <color rgba="0.8 0.8 0.8 1" />
+    </material>
+    <link name="base_link">
+        <visual>
+            <origin rpy="0 0 ${pi/2}" xyz="${frame_length/2} 0 0"/>
+            <material name="light_grey"/>
+            <geometry>
+                <mesh filename="package://robo_inspecto_launch/meshes/frame.stl" />
+            </geometry>
+        </visual>
+        <collision>
+            <origin xyz="${frame_length/2} 0 ${frame_height/2}"/>
+            <geometry>
+                <box size="${frame_length} ${frame_width} ${frame_height}" />
+            </geometry>
+        </collision>
+    </link>
 </robot>

File: robo_inspecto_launch/urdf/slede.urdf.xacro (robot description, xacro)
@@ -8,4 +8,5 @@
       height="${plate_thickness}" />
     <collision>
+      <origin xyz="0 0 ${plate_thickness/2}" />
       <geometry>
         <box size="${plate_width} ${plate_width} ${plate_thickness}" />
@@ -13,4 +14,7 @@
     </collision>
   </link>
+  <material name="dark_grey">
+    <color rgba="0.2 0.2 0.2 1" />
+  </material>
   <xacro:property name="bearing_width" value="0.065" />
   <xacro:property name="bearing_height" value="0.060" />
@@ -19,4 +23,5 @@
     <link name="${prefix}_bearing">
       <visual>
+        <material name="dark_grey"/>
         <origin rpy="${-pi/2} 0 ${pi/2}" xyz="${(bearing_width/2)} ${(-bearing_height/2)} 0" />
         <geometry>

Commit message: fixed typo

File: robo_inspecto_launch/urdf/frame.urdf.xacro (robot description, xacro)
@@ -12,5 +12,5 @@
             <material name="light_grey"/>
             <geometry>
-                <mesh filename="package://robo_inspecto_launch/meshes/frame.stl" />
+                <mesh filename="package://robo_inspecto_launch/meshes/frame.STL" />
             </geometry>
         </visual>
