Commit message: Move it update

File: robo_inspecto_launch/urdf/robot.urdf.xacro (robot description, xacro)
@@ -3,4 +3,5 @@
     <xacro:include filename="slede.urdf.xacro" />
     <xacro:include filename="frame.urdf.xacro" />
+    <xacro:property name="robot_name" value="ur5" />
     <!-- import ur5e -->
     <xacro:include filename="$(find ur_description)/urdf/ur_macro.xacro" />
@@ -9,8 +10,8 @@
         tf_prefix="ur_"
         parent="base_plate_link"
-        joint_limits_parameters_file="$(find ur_description)/config/ur5e/joint_limits.yaml"
-        kinematics_parameters_file="$(find ur_description)/config/ur5e/default_kinematics.yaml"
-        physical_parameters_file="$(find ur_description)/config/ur5e/physical_parameters.yaml"
-        visual_parameters_file="$(find ur_description)/config/ur5e/visual_parameters.yaml"
+        joint_limits_parameters_file="$(find ur_description)/config/${robot_name}/joint_limits.yaml"
+        kinematics_parameters_file="$(find ur_description)/config/${robot_name}/default_kinematics.yaml"
+        physical_parameters_file="$(find ur_description)/config/${robot_name}/physical_parameters.yaml"
+        visual_parameters_file="$(find ur_description)/config/${robot_name}/visual_parameters.yaml"
         script_filename=""
         output_recipe_filename=""
