Commit message: updated with better values

File: moveit_config/config/macro.ros2_control.xacro (robot description, xacro)
@@ -1,53 +1,24 @@
 <?xml version="1.0"?>
 <robot xmlns:xacro="http://www.ros.org/wiki/xacro">
-    <xacro:macro name="macro_ros2_control" params="name initial_positions_file">
+  <xacro:macro name="macro_ros2_control" params="
+  name
+  initial_positions_file
+  use_mock_hardware:=false
+  ">
         <xacro:property name="initial_positions" value="${load_yaml(initial_positions_file)['initial_positions']}"/>
-        <ros2_control name="${name}" type="system">
+        <ros2_control name="${name}" type="actuator">
+          <!-- check if mock -->
+          <xacro:if value="${use_mock_hardware}">
             <hardware>
                 <!-- By default, set up controllers for simulation. This won't work on real hardware -->
                 <plugin>mock_components/GenericSystem</plugin>
             </hardware>
-            <joint name="ur_shoulder_pan_joint">
-                <command_interface name="position"/>
-                <state_interface name="position">
-                  <param name="initial_value">${initial_positions['ur_shoulder_pan_joint']}</param>
-                </state_interface>
-                <state_interface name="velocity"/>
-            </joint>
-            <joint name="ur_shoulder_lift_joint">
-                <command_interface name="position"/>
-                <state_interface name="position">
-                  <param name="initial_value">${initial_positions['ur_shoulder_lift_joint']}</param>
-                </state_interface>
-                <state_interface name="velocity"/>
-            </joint>
-            <joint name="ur_elbow_joint">
-                <command_interface name="position"/>
-                <state_interface name="position">
-                  <param name="initial_value">${initial_positions['ur_elbow_joint']}</param>
-                </state_interface>
-                <state_interface name="velocity"/>
-            </joint>
-            <joint name="ur_wrist_1_joint">
-                <command_interface name="position"/>
-                <state_interface name="position">
-                  <param name="initial_value">${initial_positions['ur_wrist_1_joint']}</param>
-                </state_interface>
-                <state_interface name="velocity"/>
-            </joint>
-            <joint name="ur_wrist_2_joint">
-                <command_interface name="position"/>
-                <state_interface name="position">
-                  <param name="initial_value">${initial_positions['ur_wrist_2_joint']}</param>
-                </state_interface>
-                <state_interface name="velocity"/>
-            </joint>
-            <joint name="ur_wrist_3_joint">
-                <command_interface name="position"/>
-                <state_interface name="position">
-                  <param name="initial_value">${initial_positions['ur_wrist_3_joint']}</param>
-                </state_interface>
-                <state_interface name="velocity"/>
-            </joint>
+          </xacro:if>
+          <xacro:unless value="${use_mock_hardware}">
+            <hardware>
+                <!-- By default, set up controllers for simulation. This won't work on real hardware -->
+                <plugin>robo_inspecto_hardware/MotorHardware</plugin>
+            </hardware>
+          </xacro:unless>
             <joint name="frame_to_slede">
                 <command_interface name="position"/>
@@ -55,5 +26,4 @@
                   <param name="initial_value">${initial_positions['frame_to_slede']}</param>
                 </state_interface>
-                <state_interface name="velocity"/>
             </joint>
         </ros2_control>

File: robo_inspecto_launch/urdf/robot.urdf.xacro (robot description, xacro)
@@ -14,7 +14,9 @@
         physical_parameters_file="$(find ur_description)/config/${robot_name}/physical_parameters.yaml"
         visual_parameters_file="$(find ur_description)/config/${robot_name}/visual_parameters.yaml"
-        script_filename=""
-        output_recipe_filename=""
-        input_recipe_filename=""
+        script_filename="$(find ur_client_library)/resources/external_control.urscript"
+        output_recipe_filename="$(find ur_robot_driver)/resources/rtde_output_recipe.txt"
+        input_recipe_filename="$(find ur_robot_driver)/resources/rtde_input_recipe.txt"
+        robot_ip="192.168.10.100"
+        reverse_ip="192.168.132"
     ><origin xyz="0 0 0" rpy="0 0 0" />
     </xacro:ur_robot>
