Commit message: hope this works. otherwise fucked

File: robo_inspecto_description/urdf/frame.urdf.xacro (robot description, xacro)
@@ -12,5 +12,5 @@
             <material name="light_grey"/>
             <geometry>
-                <mesh filename="package://robo_inspecto_launch/meshes/frame.STL" />
+                <mesh filename="package://robo_inspecto_description/meshes/frame.STL" />
             </geometry>
         </visual>

File: robo_inspecto_description/urdf/macro.urdf.xacro (robot description, xacro)
@@ -2,5 +2,5 @@
 <robot xmlns:xacro="http://www.ros.org/wiki/xacro" name="macro">
     <xacro:macro name="sw_mesh_import" params="filename">
-        <mesh filename="package://robo_inspecto_launch/meshes/${filename}.STL" scale="0.001 0.001 0.001" />
+        <mesh filename="package://robo_inspecto_description/meshes/${filename}.STL" scale="0.001 0.001 0.001" />
       </xacro:macro>
       <xacro:macro name="sw_visual_import" params="filename length width height">

File: robo_inspecto_description/urdf/robot.urdf.xacro (robot description, xacro)
@@ -3,20 +3,23 @@
     <xacro:include filename="slede.urdf.xacro" />
     <xacro:include filename="frame.urdf.xacro" />
-    <xacro:property name="robot_name" value="ur5" />
     <!-- import ur5e -->
     <xacro:include filename="$(find ur_description)/urdf/ur_macro.xacro" />
+    <!-- xacro arguments -->
+    <xacro:arg name="robot_type" default="ur5"/>
+    <xacro:arg name="robot_ip" default=""/>
+    <xacro:arg name="reverse_ip" default="0.0.0.0"/>
     <xacro:ur_robot
         name="ur"
         tf_prefix="ur_"
         parent="base_plate_link"
-        joint_limits_parameters_file="$(find ur_description)/config/${robot_name}/joint_limits.yaml"
-        kinematics_parameters_file="$(find ur_description)/config/${robot_name}/default_kinematics.yaml"
-        physical_parameters_file="$(find ur_description)/config/${robot_name}/physical_parameters.yaml"
-        visual_parameters_file="$(find ur_description)/config/${robot_name}/visual_parameters.yaml"
+        joint_limits_parameters_file="$(find ur_description)/config/$(arg robot_type)/joint_limits.yaml"
+        kinematics_parameters_file="$(find ur_description)/config/$(arg robot_type)/default_kinematics.yaml"
+        physical_parameters_file="$(find ur_description)/config/$(arg robot_type)/physical_parameters.yaml"
+        visual_parameters_file="$(find ur_description)/config/$(arg robot_type)/visual_parameters.yaml"
         script_filename="$(find ur_client_library)/resources/external_control.urscript"
         output_recipe_filename="$(find ur_robot_driver)/resources/rtde_output_recipe.txt"
         input_recipe_filename="$(find ur_robot_driver)/resources/rtde_input_recipe.txt"
-        robot_ip="192.168.10.100"
-        reverse_ip="192.168.132"
+        robot_ip="$(arg robot_ip)"
+        reverse_ip="$(arg reverse_ip)"
     ><origin xyz="0 0 0" rpy="0 0 0" />
     </xacro:ur_robot>

File: robo_inspecto_moveit_config/config/macro.urdf.xacro (robot description, xacro)
@@ -3,5 +3,5 @@
     <xacro:arg name="initial_positions_file" default="initial_positions.yaml" />
     <!-- Import macro urdf file -->
-    <xacro:include filename="$(find robo_inspecto_launch)/urdf/robot.urdf.xacro" />
+    <xacro:include filename="$(find robo_inspecto_description)/urdf/robot.urdf.xacro" />
     <!-- Import control_xacro -->
     <xacro:include filename="macro.ros2_control.xacro" />
